File: F4Dev.sch (KiCad schematic (older format))
At the start: 65 parts, among them J1 USB_MINI, P1 CONN_12X2, P2 CONN_12X2, P3 CONN_13X2, P4 CONN_13X2, P5 CONN_6, SW1 SW_PUSH_SMALL_4_PINS, U1 STM32F407VG, U2 BT0417C, U3 FT230XS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

Commit message: Now L3G4200D can also be used as gyroscope.
Parts:
- added C38: 470n, symbol C
- added R6: 10k, symbol R
- U5: value L3GD20 -> L3GD20/L3G4200D
Other:
- note added: "GYROSCOPE\n(0b1101011\n 0b1101001)"
- note added: "L3G4200D ONLY"
- note removed: "GYROSCOPE\n(0b1101011)"
- moved on the sheet: C25, C26, C28, U5
